File: PCB-KiCAD/TeensyRPN42/TeensyRPN42.kicad_pcb (KiCad board)
At the start: 2 copper layers, 47 parts, among them SW1 SW_DPST_x2, SW10 SW_DPST_x2, SW11 SW_DPST_x2, SW12 SW_DPST_x2, SW13 SW_DPST_x2, SW14 SW_DPST_x2, SW15 SW_DPST_x2, SW16 SW_DPST_x2, SW17 SW_DPST_x2, SW18 SW_DPST_x2, SW19 SW_DPST_x2, SW2 SW_DPST_x2, SW20 SW_DPST_x2, SW21 SW_DPST_x2, SW22 SW_DPST_x2, SW23 SW_DPST_x2, SW24 SW_DPST_x2, SW25 SW_DPST_x2, SW26 SW_DPST_x2, SW27 SW_DPST_x2, SW28 SW_DPST_x2, SW29 SW_DPST_x2, SW3 SW_DPST_x2, SW30 SW_DPST_x2, SW31 SW_DPST_x2, SW32 SW_DPST_x2, SW33 SW_DPST_x2, SW34 SW_DPST_x2, SW35 SW_DPST_x2, SW36 SW_DPST_x2, SW37 SW_DPST_x2, SW4 SW_DPST_x2, SW5 SW_DPST_x2, SW6 SW_DPST_x2, SW7 SW_DPST_x2, SW8 SW_DPST_x2, SW9 SW_DPST_x2, U1 74HC165, U2 74HC165, U3 74HC165, U4 74HC165, U5 74HC165

Commit message: Added KeyChoc stuff
Parts:
- added SW38: SW_DPST_x2, keyswitches:Kailh_socket_PG1350, F.Cu at (182.8, 42.8)
- added SW39: SW_DPST_x2, keyswitches:Kailh_socket_PG1350, F.Cu at (182.8, 59.6)
- added SW40: SW_DPST_x2, keyswitches:Kailh_socket_PG1350, F.Cu at (182.8, 76.5)
- added SW41: SW_DPST_x2, keyswitches:Kailh_socket_PG1350, F.Cu at (182.8, 93.3)
- added SW42: SW_DPST_x2, keyswitches:Kailh_socket_PG1350, F.Cu at (182.8, 110.2)
- added SW43: SW_DPST_x2, keyswitches:Kailh_socket_PG1350, F.Cu at (182.8, 127.0)
- added SW44: SW_DPST_x2, keyswitches:Kailh_socket_PG1350, F.Cu at (182.8, 143.8)
- added SW45: SW_DPST_x2, keyswitches:Kailh_socket_PG1350, F.Cu at (200.9, 42.8)
- added SW46: SW_DPST_x2, keyswitches:Kailh_socket_PG1350, F.Cu at (200.9, 59.6)
- added SW48: SW_DPST_x2, keyswitches:Kailh_socket_PG1350, F.Cu at (200.9, 76.5)
- added SW49: SW_DPST_x2, keyswitches:Kailh_socket_PG1350, F.Cu at (200.9, 93.3)
- added SW50: SW_DPST_x2, keyswitches:Kailh_socket_PG1350, F.Cu at (200.9, 110.2)
- added SW51: SW_DPST_x2, keyswitches:Kailh_socket_PG1350, F.Cu at (200.9, 127.0)
- added SW52: SW_DPST_x2, keyswitches:Kailh_socket_PG1350, F.Cu at (200.9, 143.8)
- added SW53: SW_DPST_x2, keyswitches:Kailh_socket_PG1350, F.Cu at (219.1, 42.8)
- added SW54: SW_DPST_x2, keyswitches:Kailh_socket_PG1350, F.Cu at (219.1, 59.6)
- added SW55: SW_DPST_x2, keyswitches:Kailh_socket_PG1350, F.Cu at (219.1, 76.5)
- added SW56: SW_DPST_x2, keyswitches:Kailh_socket_PG1350, F.Cu at (219.1, 93.3)
- added SW57: SW_DPST_x2, keyswitches:Kailh_socket_PG1350, F.Cu at (219.1, 110.2)
- added SW58: SW_DPST_x2, keyswitches:Kailh_socket_PG1350, F.Cu at (219.1, 127.0)
- added SW59: SW_DPST_x2, keyswitches:Kailh_socket_PG1350, F.Cu at (219.1, 143.8)
- added SW60: SW_DPST_x2, keyswitches:Kailh_socket_PG1350, F.Cu at (237.2, 42.8)
- added SW61: SW_DPST_x2, keyswitches:Kailh_socket_PG1350, F.Cu at (237.2, 59.6)
- added SW62: SW_DPST_x2, keyswitches:Kailh_socket_PG1350, F.Cu at (237.2, 76.5)
- added SW63: SW_DPST_x2, keyswitches:Kailh_socket_PG1350, F.Cu at (237.2, 93.3)
- added SW64: SW_DPST_x2, keyswitches:Kailh_socket_PG1350, F.Cu at (237.2, 110.2)
- added SW65: SW_DPST_x2, keyswitches:Kailh_socket_PG1350, F.Cu at (237.2, 127.0)
- added SW66: SW_DPST_x2, keyswitches:Kailh_socket_PG1350, F.Cu at (237.2, 143.8)
- added SW67: SW_DPST_x2, keyswitches:Kailh_socket_PG1350, F.Cu at (255.3, 42.8)
- added SW68: SW_DPST_x2, keyswitches:Kailh_socket_PG1350, F.Cu at (255.3, 59.6)
- added SW69: SW_DPST_x2, keyswitches:Kailh_socket_PG1350, F.Cu at (255.3, 76.5)
- added SW70: SW_DPST_x2, keyswitches:Kailh_socket_PG1350, F.Cu at (255.3, 93.3)
- added SW71: SW_DPST_x2, keyswitches:Kailh_socket_PG1350, F.Cu at (255.3, 110.2)
- added SW72: SW_DPST_x2, keyswitches:Kailh_socket_PG1350, F.Cu at (255.3, 127.0)
- added SW73: SW_DPST_x2, keyswitches:Kailh_socket_PG1350, F.Cu at (255.3, 143.8)
- added SW74: SW_DPST_x2, keyswitches:Kailh_socket_PG1350, F.Cu at (273.5, 42.8)
- added SW75: SW_DPST_x2, keyswitches:Kailh_socket_PG1350, F.Cu at (273.5, 59.6)
- added SW76: SW_DPST_x2, keyswitches:Kailh_socket_PG1350, F.Cu at (273.5, 76.5)
- added SW77: SW_DPST_x2, keyswitches:Kailh_socket_PG1350, F.Cu at (273.5, 93.3)
- added SW78: SW_DPST_x2, keyswitches:Kailh_socket_PG1350, F.Cu at (273.5, 110.2)
- added SW79: SW_DPST_x2, keyswitches:Kailh_socket_PG1350, F.Cu at (273.5, 127.0)
- moved U2 35.0 mm to (156.4, 107.3)
- moved U3 35.0 mm to (146.2, 107.3)
- moved U4 35.0 mm to (136.1, 107.3)
- moved U5 35.0 mm to (125.7, 107.1)
- moved U1 35.0 mm to (166.6, 107.3)
- moved RN4 23.7 mm to (132.8, 88.2)
- moved RN1 23.7 mm to (132.8, 75.1)
- moved RN2 23.7 mm to (132.8, 79.5)
- moved RN3 23.7 mm to (132.8, 83.8)
- moved RN5 23.7 mm to (132.8, 92.5)
Other:
- board outline added: 113 x 133 mm

Commit message: A little PCBing
Parts:
- removed RN1, RN2, RN3, RN4, RN5: R_Network08, Resistor_THT:R_Array_SIP9
- removed SW1, SW10, SW11, SW12, SW13, SW14, SW15, SW16, SW17, SW18, SW19, SW2, SW20, SW21, SW22, SW23, SW24, SW25, SW26, SW27, SW28, SW29, SW3, SW30, SW31, SW32, SW33, SW34, SW35, SW36, SW37, SW4, SW5, SW6, SW7, SW8, SW9: SW_DPST_x2, RPN42Library:swith12mm
- removed SW59, SW66, SW73, SW79: SW_DPST_x2, keyswitches:Kailh_socket_PG1350
- removed U3, U4, U5: 74HC165, Package_SO:SOIC-16W_5.3x10.2mm_P1.27mm
- added D1: SK6812MINI, LED_SMD:LED_SK6812MINI_PLCC4_3.5x3.5mm_P1.75mm, F.Cu at (87.8, 60.9)
- added D2: SK6805, LED_SMD:LED_SK6805_PLCC4_2.4x2.7mm_P1.3mm, F.Cu at (86.9, 65.4)
- added DS1: OLED-128O064D, Display:OLED-128O064D, F.Cu at (134.9, 93.5)
- SW38, SW39, SW40, SW41, SW42, SW43, SW44, SW45, SW48, SW49, SW50, SW51, SW52, SW58, SW61, SW62, SW63, SW64, SW65, SW68, SW69, SW70, SW71, SW72, SW75, SW76, SW77, SW78: footprint keyswitches:Kailh_socket_PG1350 -> PCM_Switch_Keyboard_Kailh:SW_Kailh_Choc_V1_1.00u
- SW46: footprint keyswitches:Kailh_socket_PG1350 -> PCM_Switch_Keyboard_Kailh:SW_Kailh_Choc_V1_2.00u
- SW53, SW54, SW55, SW56, SW57, SW60, SW67, SW74: footprint keyswitches:Kailh_socket_PG1350 -> PCM_Switch_Keyboard_Kailh:SW_Kailh_Choc_V1_1.25u
- U1: value 74HC165 -> HT1632C-52LQFP; footprint Package_SO:SOIC-16W_5.3x10.2mm_P1.27mm -> Package_QFP:LQFP-52_14x14mm_P1mm; moved to F.Cu
- U2: value 74HC165 -> STM32F411RETx; footprint Package_SO:SOIC-16W_5.3x10.2mm_P1.27mm -> Package_QFP:LQFP-64_10x10mm_P0.5mm; moved to F.Cu
- moved SW74 284.2 mm to (58.3, 228.4), turned to 180 degrees
- moved SW67 258.0 mm to (58.3, 209.4), turned to 180 degrees
- moved SW75 256.3 mm to (76.6, 223.6), turned to 180 degrees
- moved SW76 233.9 mm to (92.2, 224.2), turned to 180 degrees
- moved SW60 232.2 mm to (58.2, 190.6), turned to 180 degrees
- moved SW69 222.3 mm to (75.2, 206.7), turned to 180 degrees
- moved SW77 209.4 mm to (109.7, 223.8), turned to 180 degrees
- moved SW61 208.3 mm to (73.7, 188.7), turned to 180 degrees
- moved SW53 206.2 mm to (58.3, 171.8), turned to 180 degrees
- moved SW70 199.0 mm to (91.7, 206.5), turned to 180 degrees
- moved SW62 183.6 mm to (91.7, 188.4), turned to 180 degrees
- moved SW54 178.0 mm to (80.9, 171.8), turned to 180 degrees
- moved SW71 174.5 mm to (109.5, 205.9), turned to 180 degrees
- moved SW78 173.2 mm to (144.8, 226.0), turned to 180 degrees
- moved SW46 163.7 mm to (65.7, 151.9), turned to 180 degrees
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Connections:
- U1 pad 11: Net-(RN1-R1) -> unconnected-(U1-ROW2-Pad11)
- U1 pad 12: Net-(RN1-R2) -> unconnected-(U1-ROW1-Pad12)
- U1 pad 13: Net-(RN1-R3) -> unconnected-(U1-ROW0-Pad13)
- U1 pad 14: Net-(RN1-R4) -> Net-(U1-VSS-Pad14)
- U1 pad 3: Net-(RN1-R5) -> unconnected-(U1-ROW9-Pad3)
- U1 pad 4: Net-(RN1-R6) -> unconnected-(U1-ROW8-Pad4)
- U1 pad 5: Net-(RN1-R7) -> unconnected-(U1-ROW7-Pad5)
- U1 pad 6: Net-(RN1-R8) -> unconnected-(U1-ROW6-Pad6)
Other:
- board size 113 x 133 mm -> 113 x 198.3 mm

Commit message: more PCB
Parts:
- removed DS1: OLED-128O064D, Display:OLED-128O064D
- added C1: 20pF, Capacitor_SMD:C_0603_1608Metric_Pad1.08x0.95mm_HandSolder, F.Cu at (109.0, 88.6)
- added C10: 100nF, Capacitor_SMD:C_0603_1608Metric_Pad1.08x0.95mm_HandSolder, F.Cu at (126.3, 90.5)
- added C11: 100nF, Capacitor_SMD:C_0603_1608Metric_Pad1.08x0.95mm_HandSolder, F.Cu at (128.8, 90.5)
- added C12: 100nF, Capacitor_SMD:C_0603_1608Metric_Pad1.08x0.95mm_HandSolder, F.Cu at (131.3, 90.5)
- added C13: 100nF, Capacitor_SMD:C_0603_1608Metric_Pad1.08x0.95mm_HandSolder, F.Cu at (139.8, 81.8)
- added C14: 100nF, Capacitor_SMD:C_0603_1608Metric_Pad1.08x0.95mm_HandSolder, B.Cu at (66.1, 116.8)
- added C15: 100nF, Capacitor_SMD:C_0603_1608Metric_Pad1.08x0.95mm_HandSolder, B.Cu at (84.9, 116.3)
- added C16: 100nF, Capacitor_SMD:C_0603_1608Metric_Pad1.08x0.95mm_HandSolder, B.Cu at (122.2, 116.2)
- added C17: 100nF, Capacitor_SMD:C_0603_1608Metric_Pad1.08x0.95mm_HandSolder, B.Cu at (140.9, 116.6)
- added C18: 100nF, Capacitor_SMD:C_0603_1608Metric_Pad1.08x0.95mm_HandSolder, B.Cu at (65.9, 135.6)
- added C19: 100nF, Capacitor_SMD:C_0603_1608Metric_Pad1.08x0.95mm_HandSolder, B.Cu at (84.7, 135.4)
- added C2: 20pF, Capacitor_SMD:C_0603_1608Metric_Pad1.08x0.95mm_HandSolder, F.Cu at (96.4, 88.6)
- added C20: 100nF, Capacitor_SMD:C_0603_1608Metric_Pad1.08x0.95mm_HandSolder, B.Cu at (122.2, 135.3)
- added C21: 100nF, Capacitor_SMD:C_0603_1608Metric_Pad1.08x0.95mm_HandSolder, B.Cu at (140.9, 135.6)
- added C22: 100nF, Capacitor_SMD:C_0603_1608Metric_Pad1.08x0.95mm_HandSolder, B.Cu at (56.4, 155.7)
- added C23: 100nF, Capacitor_SMD:C_0603_1608Metric_Pad1.08x0.95mm_HandSolder, B.Cu at (81.0, 155.4)
- added C24: 100nF, Capacitor_SMD:C_0603_1608Metric_Pad1.08x0.95mm_HandSolder, B.Cu at (122.4, 155.2)
- added C25: 100nF, Capacitor_SMD:C_0603_1608Metric_Pad1.08x0.95mm_HandSolder, B.Cu at (141.1, 155.4)
- added C3: 100nF, Capacitor_SMD:C_0603_1608Metric_Pad1.08x0.95mm_HandSolder, F.Cu at (57.9, 89.3)
- added C4: 10u, Capacitor_SMD:C_1206_3216Metric_Pad1.33x1.80mm_HandSolder, F.Cu at (85.0, 90.7)
- added C5: 10u, Capacitor_SMD:C_1206_3216Metric_Pad1.33x1.80mm_HandSolder, F.Cu at (85.0, 94.1)
- added C6: 100nF, Capacitor_SMD:C_0603_1608Metric_Pad1.08x0.95mm_HandSolder, F.Cu at (90.2, 90.3)
- added C7: 100nF, Capacitor_SMD:C_0603_1608Metric_Pad1.08x0.95mm_HandSolder, F.Cu at (118.7, 90.5)
- added C8: 100nF, Capacitor_SMD:C_0603_1608Metric_Pad1.08x0.95mm_HandSolder, F.Cu at (121.2, 90.5)
- added C9: 100nF, Capacitor_SMD:C_0603_1608Metric_Pad1.08x0.95mm_HandSolder, F.Cu at (123.8, 90.5)
- added D10: SK6805, LED_SMD:LED_SK6805_PLCC4_2.4x2.7mm_P1.3mm, F.Cu at (112.9, 135.3)
- added D11: SK6805, LED_SMD:LED_SK6805_PLCC4_2.4x2.7mm_P1.3mm, F.Cu at (131.7, 135.3)
- added D12: SK6805, LED_SMD:LED_SK6805_PLCC4_2.4x2.7mm_P1.3mm, F.Cu at (150.4, 135.3)
- added D13: SK6805, LED_SMD:LED_SK6805_PLCC4_2.4x2.7mm_P1.3mm, F.Cu at (51.0, 159.9)
- added D14: SK6805, LED_SMD:LED_SK6805_PLCC4_2.4x2.7mm_P1.3mm, F.Cu at (65.7, 155.3)
- added D15: SK6805, LED_SMD:LED_SK6805_PLCC4_2.4x2.7mm_P1.3mm, F.Cu at (94.2, 155.3)
- added D16: SK6805, LED_SMD:LED_SK6805_PLCC4_2.4x2.7mm_P1.3mm, F.Cu at (113.0, 155.3)
- added D17: SK6805, LED_SMD:LED_SK6805_PLCC4_2.4x2.7mm_P1.3mm, F.Cu at (131.8, 155.3)
- added D18: SK6805, LED_SMD:LED_SK6805_PLCC4_2.4x2.7mm_P1.3mm, F.Cu at (150.4, 155.3)
- added D3: SK6805, LED_SMD:LED_SK6805_PLCC4_2.4x2.7mm_P1.3mm, F.Cu at (94.3, 115.3)
- added D4: SK6805, LED_SMD:LED_SK6805_PLCC4_2.4x2.7mm_P1.3mm, F.Cu at (112.9, 115.3)
- added D5: SK6805, LED_SMD:LED_SK6805_PLCC4_2.4x2.7mm_P1.3mm, F.Cu at (131.7, 115.3)
- added D6: SK6805, LED_SMD:LED_SK6805_PLCC4_2.4x2.7mm_P1.3mm, F.Cu at (150.4, 115.3)
- added D7: SK6805, LED_SMD:LED_SK6805_PLCC4_2.4x2.7mm_P1.3mm, F.Cu at (56.7, 135.3)
- added D8: SK6805, LED_SMD:LED_SK6805_PLCC4_2.4x2.7mm_P1.3mm, F.Cu at (75.5, 135.3)
- added D9: SK6805, LED_SMD:LED_SK6805_PLCC4_2.4x2.7mm_P1.3mm, F.Cu at (94.3, 135.3)
- added H1: MountingHole, MountingHole:MountingHole_3.2mm_M3_ISO7380, F.Cu at (57.9, 78.5)
- added H2: MountingHole, MountingHole:MountingHole_3.2mm_M3_ISO7380, F.Cu at (57.9, 105.9)
- added H3: MountingHole, MountingHole:MountingHole_3.2mm_M3_ISO7380, F.Cu at (149.4, 78.5)
- added H4: MountingHole, MountingHole:MountingHole_3.2mm_M3_ISO7380, F.Cu at (149.4, 105.9)
- added J1: Conn_01x06, Connector_PinHeader_2.54mm:PinHeader_1x06_P2.54mm_Vertical, B.Cu at (81.5, 78.2)
- added J2: Conn_01x04, Connector_PinSocket_2.54mm:PinSocket_1x04_P2.54mm_Vertical, F.Cu at (155.2, 88.9)
- added J3: Conn_02x08_Odd_Even, RPN42Library:OLED-2.8inch16pin, B.Cu at (103.7, 92.2)
- added L1: L_Ferrite_Small, Inductor_SMD:L_0603_1608Metric_Pad1.05x0.95mm_HandSolder, F.Cu at (90.2, 92.8)
- added L2: L_Ferrite_Small, Inductor_SMD:L_0603_1608Metric_Pad1.05x0.95mm_HandSolder, F.Cu at (140.2, 85.3)
- added L3: L_Ferrite_Small, Inductor_SMD:L_0603_1608Metric_Pad1.05x0.95mm_HandSolder, F.Cu at (49.5, 108.2)
- added R1: 10k, Resistor_SMD:R_0603_1608Metric_Pad0.98x0.95mm_HandSolder, F.Cu at (68.6, 96.4)
- added R2: 330, Resistor_SMD:R_0603_1608Metric_Pad0.98x0.95mm_HandSolder, F.Cu at (51.6, 108.2)
- added R3: 2.2k, Resistor_SMD:R_0603_1608Metric_Pad0.98x0.95mm_HandSolder, F.Cu at (133.8, 90.5)
- added R4: 2.2k, Resistor_SMD:R_0603_1608Metric_Pad0.98x0.95mm_HandSolder, F.Cu at (136.3, 90.5)
- added R5: 10k, Resistor_SMD:R_0603_1608Metric_Pad0.98x0.95mm_HandSolder, F.Cu at (57.9, 85.3)
- added SW1: SW_Push_Dual, Button_Switch_SMD:SW_SPST_EVQQ2, F.Cu at (50.8, 84.8)
- added SW2: SW_Push_Dual, Button_Switch_SMD:SW_SPST_EVQQ2, F.Cu at (50.8, 97.5)
- added U3: SN74LV1T125DBV, Package_TO_SOT_SMD:SOT-23-5, F.Cu at (66.5, 106.2)
- added Y1: Crystal 8MHz, Crystal:Crystal_SMD_HC49-SD_HandSoldering, F.Cu at (102.4, 83.6)
- D1: value SK6812MINI -> SK6805; footprint LED_SMD:LED_SK6812MINI_PLCC4_3.5x3.5mm_P1.75mm -> LED_SMD:LED_SK6805_PLCC4_2.4x2.7mm_P1.3mm
- SW61, SW62, SW63, SW64, SW69, SW70, SW71, SW72, SW75, SW76, SW77, SW78: footprint PCM_Switch_Keyboard_Kailh:SW_Kailh_Choc_V1_1.00u -> PCM_Switch_Keyboard_Kailh:SW_Kailh_Choc_V1_1.25u
- U1: value HT1632C-52LQFP -> AMS1117-3.3; footprint Package_QFP:LQFP-52_14x14mm_P1mm -> Package_TO_SOT_SMD:SOT-223-3_TabPin2
- moved D1 62.6 mm to (56.8, 115.3), turned to 180 degrees
- moved D2 51.2 mm to (75.5, 115.3), turned to 180 degrees
- moved SW77 49.0 mm to (126.1, 270.0)
- moved SW76 47.1 mm to (103.5, 270.0)
- moved SW71 47.1 mm to (126.1, 250.0)
- moved SW75 46.6 mm to (80.9, 270.0)
- moved SW63 45.3 mm to (126.1, 230.0)
- moved SW70 45.1 mm to (103.5, 250.0)
- moved SW78 44.2 mm to (148.6, 270.0)
- moved SW69 43.7 mm to (80.9, 250.0)
- moved SW62 43.2 mm to (103.5, 230.0)
- moved SW72 42.2 mm to (148.5, 250.0)
- moved SW61 42.0 mm to (80.9, 230.0)
- moved SW74 41.6 mm to (58.3, 270.0)
- moved SW67 40.6 mm to (58.3, 250.0)
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Connections:
- D1 pad 1: unconnected-(D1-DOUT-Pad1) -> Net-(D1-DOUT)
- D1 pad 2: unconnected-(D1-VSS-Pad2) -> GND
- D1 pad 3: unconnected-(D1-DIN-Pad3) -> Net-(D1-DIN)
- D1 pad 4: unconnected-(D1-VDD-Pad4) -> /LEDS/V-LED
- D2 pad 1: unconnected-(D2-DOUT-Pad1) -> Net-(D2-DOUT)
- D2 pad 2: unconnected-(D2-VSS-Pad2) -> GND
- D2 pad 3: unconnected-(D2-DIN-Pad3) -> Net-(D1-DOUT)
- D2 pad 4: unconnected-(D2-VDD-Pad4) -> /LEDS/V-LED
- SW38 pad 1: unconnected-(SW38A-A-Pad1) -> ROW1
- SW38 pad 2: unconnected-(SW38A-B-Pad2) -> COL0
- SW39 pad 1: unconnected-(SW39A-A-Pad1) -> ROW2
- SW40 pad 1: unconnected-(SW40A-A-Pad1) -> ROW2
- SW41 pad 1: unconnected-(SW41A-A-Pad1) -> ROW2
- SW42 pad 1: unconnected-(SW42A-A-Pad1) -> ROW2
- SW43 pad 1: unconnected-(SW43A-A-Pad1) -> ROW2
- SW44 pad 1: unconnected-(SW44A-A-Pad1) -> ROW2
- SW45 pad 1: unconnected-(SW45A-A-Pad1) -> ROW1
- SW45 pad 2: unconnected-(SW45A-B-Pad2) -> COL1
- SW46 pad 1: unconnected-(SW46A-A-Pad1) -> ROW3
- SW48 pad 1: unconnected-(SW48A-A-Pad1) -> ROW3
- SW49 pad 1: unconnected-(SW49A-A-Pad1) -> ROW3
- SW50 pad 1: unconnected-(SW50A-A-Pad1) -> ROW3
- SW51 pad 1: unconnected-(SW51A-A-Pad1) -> ROW1
- SW51 pad 2: unconnected-(SW51A-B-Pad2) -> COL2
- SW52 pad 1: unconnected-(SW52A-A-Pad1) -> ROW3
- SW53 pad 1: unconnected-(SW53A-A-Pad1) -> ROW4
- SW54 pad 1: unconnected-(SW54A-A-Pad1) -> ROW4
- SW55 pad 1: unconnected-(SW55A-A-Pad1) -> ROW4
- SW56 pad 1: unconnected-(SW56A-A-Pad1) -> ROW4
- SW57 pad 1: unconnected-(SW57A-A-Pad1) -> ROW4
- SW58 pad 1: unconnected-(SW58A-A-Pad1) -> ROW1
- SW58 pad 2: unconnected-(SW58A-B-Pad2) -> COL3
- SW60 pad 1: unconnected-(SW60A-A-Pad1) -> ROW5
- SW61 pad 1: unconnected-(SW61A-A-Pad1) -> ROW5
- SW62 pad 1: unconnected-(SW62A-A-Pad1) -> ROW5
- SW63 pad 1: unconnected-(SW63A-A-Pad1) -> ROW5
- SW64 pad 1: unconnected-(SW64A-A-Pad1) -> ROW5
- SW65 pad 1: unconnected-(SW65A-A-Pad1) -> ROW1
- SW65 pad 2: unconnected-(SW65A-B-Pad2) -> COL4
- SW67 pad 1: unconnected-(SW67A-A-Pad1) -> ROW6
- SW68 pad 1: unconnected-(SW68A-A-Pad1) -> ROW1
- SW68 pad 2: unconnected-(SW68A-B-Pad2) -> COL5
- SW69 pad 1: unconnected-(SW69A-A-Pad1) -> ROW6
- SW70 pad 1: unconnected-(SW70A-A-Pad1) -> ROW6
- SW71 pad 1: unconnected-(SW71A-A-Pad1) -> ROW6
- SW72 pad 1: unconnected-(SW72A-A-Pad1) -> ROW6
- SW74 pad 1: unconnected-(SW74A-A-Pad1) -> ROW7
- SW75 pad 1: unconnected-(SW75A-A-Pad1) -> ROW7
- SW76 pad 1: unconnected-(SW76A-A-Pad1) -> ROW7
- SW77 pad 1: unconnected-(SW77A-A-Pad1) -> ROW7
- SW78 pad 1: unconnected-(SW78A-A-Pad1) -> ROW7
- U1 pad 1: unconnected-(U1-ROW11-Pad1) -> GND
- U1 pad 2: unconnected-(U1-ROW10-Pad2) -> +3.3V
- U1 pad 3: unconnected-(U1-ROW9-Pad3) -> /VIN
- U2 pad 12: unconnected-(U2-VSSA-Pad12) -> GND
- U2 pad 13: unconnected-(U2-VDDA-Pad13) -> Net-(U2-VDDA)
- U2 pad 16: unconnected-(U2-PA2-Pad16) -> /USAR_TX
- U2 pad 17: unconnected-(U2-PA3-Pad17) -> /USART_RX
- U2 pad 18: Net-(U2-VSS-Pad18) -> GND
- U2 pad 19: unconnected-(U2-VDD-Pad19) -> +3.3V
- U2 pad 20: unconnected-(U2-PA4-Pad20) -> /OLED_CS
- U2 pad 21: unconnected-(U2-PA5-Pad21) -> /SCK1
- U2 pad 22: unconnected-(U2-PA6-Pad22) -> /MISO1
- U2 pad 23: unconnected-(U2-PA7-Pad23) -> /MOSI1
- U2 pad 29: unconnected-(U2-PB10-Pad29) -> LEDs
- U2 pad 31: Net-(U2-VSS-Pad18) -> GND
- U2 pad 32: unconnected-(U2-VDD-Pad32) -> +3.3V
- U2 pad 38: unconnected-(U2-PC7-Pad38) -> COL0
- U2 pad 39: unconnected-(U2-PC8-Pad39) -> COL1
- U2 pad 40: unconnected-(U2-PC9-Pad40) -> COL2
- U2 pad 41: unconnected-(U2-PA8-Pad41) -> ROW0
- U2 pad 42: unconnected-(U2-PA9-Pad42) -> ROW1
- U2 pad 43: unconnected-(U2-PA10-Pad43) -> ROW2
- U2 pad 44: unconnected-(U2-PA11-Pad44) -> ROW3
- U2 pad 45: unconnected-(U2-PA12-Pad45) -> ROW4
- U2 pad 46: unconnected-(U2-PA13-Pad46) -> ROW5
- U2 pad 47: Net-(U2-VSS-Pad18) -> GND
- U2 pad 48: unconnected-(U2-VDD-Pad48) -> +3.3V
- U2 pad 49: unconnected-(U2-PA14-Pad49) -> ROW6
- U2 pad 5: unconnected-(U2-PH0-Pad5) -> Net-(U2-PH0)
- U2 pad 50: unconnected-(U2-PA15-Pad50) -> ROW7
- U2 pad 51: unconnected-(U2-PC10-Pad51) -> COL3
- U2 pad 52: unconnected-(U2-PC11-Pad52) -> COL4
- U2 pad 53: unconnected-(U2-PC12-Pad53) -> COL5
- U2 pad 55: unconnected-(U2-PB3-Pad55) -> /SWO
- U2 pad 6: unconnected-(U2-PH1-Pad6) -> Net-(U2-PH1)
- U2 pad 60: unconnected-(U2-BOOT0-Pad60) -> Net-(U2-BOOT0)
- U2 pad 61: unconnected-(U2-PB8-Pad61) -> /SCL1
- U2 pad 62: unconnected-(U2-PB9-Pad62) -> /SDA1
- U2 pad 63: Net-(U2-VSS-Pad18) -> GND
- U2 pad 64: unconnected-(U2-VDD-Pad64) -> +3.3V
- U2 pad 7: unconnected-(U2-NRST-Pad7) -> /NRST
Routing:
- net /LEDS/V-LED: track 0.00 -> 456.3 mm, vias 0 -> 12
- net ROW1: track 0.00 -> 171.7 mm, vias 0 -> 1
- net ROW2: track 0.00 -> 163.8 mm, vias 0 -> 2
- net ROW3: track 0.00 -> 154.6 mm, vias 0 -> 2
- net Net-(D12-DOUT): track 0.00 -> 120.3 mm
- net unconnected-(D18-DOUT-Pad1): track 0.00 -> 116.7 mm
- net Net-(D6-DOUT): track 0.00 -> 113.3 mm
- net COL5: track 0.00 -> 105.6 mm, vias 0 -> 1
- net COL4: track 0.00 -> 86.0 mm, vias 0 -> 1
- net COL3: track 0.00 -> 78.2 mm, vias 0 -> 1
- net ROW7: track 0.00 -> 75.6 mm, vias 0 -> 1
- net ROW6: track 0.00 -> 74.3 mm, vias 0 -> 1
- net ROW4: track 0.00 -> 70.6 mm, vias 0 -> 1
- net ROW5: track 0.00 -> 70.0 mm, vias 0 -> 1
- net COL0: track 0.00 -> 65.5 mm, vias 0 -> 1
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- added copper zone on B.Cu, net GND
- added copper zone on F.Cu, net GND
Other:
- board size 113 x 198.3 mm -> 113 x 101.1 mm
- board text added: "RESET"

Commit message: more pcb ...
Parts:
- removed U1: AMS1117-3.3, Package_TO_SOT_SMD:SOT-223-3_TabPin2
- added C26: 1nF, Capacitor_SMD:C_0603_1608Metric_Pad1.08x0.95mm_HandSolder, F.Cu at (132.4, 83.3)
- added J4: Serial, Connector_PinHeader_2.54mm:PinHeader_1x03_P2.54mm_Vertical, B.Cu at (88.4, 78.2)
- added J5: Bat JST, Connector_JST:JST_EH_S2B-EH_1x02_P2.50mm_Horizontal, F.Cu at (119.6, 79.0)
- added U4: MCP1727-3302xSN, Package_SO:SOIC-8_3.9x4.9mm_P1.27mm, F.Cu at (134.4, 78.9)
- added Y3: Crystal_GND24, Crystal:Crystal_SMD_0603-4Pin_6.0x3.5mm_HandSoldering, F.Cu at (102.7, 88.7)
- J1: value Conn_01x06 -> SWD
- SW1, SW2: moved to B.Cu
- U2: value STM32F411RETx -> STM32F405RGTx
- U3: value SN74LV1T125DBV -> 74!AHCT!125; footprint Package_TO_SOT_SMD:SOT-23-5 -> Package_TO_SOT_SMD:SOT-353_SC-70-5
- moved C4 43.1 mm to (127.5, 83.3), turned to 90 degrees
- moved C5 33.0 mm to (117.3, 87.6)
- moved C8 31.0 mm to (95.1, 107.2), turned to 180 degrees
- moved SW53 27.4 mm to (58.3, 182.6)
- moved SW54 27.4 mm to (80.9, 182.6)
- moved SW55 27.4 mm to (103.5, 182.6)
- moved SW56 27.4 mm to (126.1, 182.6)
- moved SW57 27.4 mm to (148.7, 182.6)
- moved SW60 27.4 mm to (58.3, 202.6)
- moved SW61 27.4 mm to (80.9, 202.6)
- moved SW62 27.4 mm to (103.5, 202.6)
- moved SW63 27.4 mm to (126.2, 202.6)
- moved SW64 27.4 mm to (148.7, 202.6)
- moved SW67 27.4 mm to (58.4, 222.6)
- moved SW69 27.4 mm to (80.9, 222.6)
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Connections:
- C6 pad 1: Net-(U2-VDDA) -> /VDDA
- C6 pad 2: Net-(U2-VDDA) -> GND
- J1 pad 2: unconnected-(J1-Pin_2-Pad2) -> /TCK
- J1 pad 3: unconnected-(J1-Pin_3-Pad3) -> GND
- J1 pad 4: unconnected-(J1-Pin_4-Pad4) -> /TMS
- J1 pad 5: unconnected-(J1-Pin_5-Pad5) -> /NRST
- J1 pad 6: unconnected-(J1-Pin_6-Pad6) -> /SWO
- L1 pad 2: Net-(U2-VDDA) -> /VDDA
- SW2 pad 1: Net-(SW2-Pad1) -> GND
- U2 pad 12: GND -> unconnected-(U2-VSSA-Pad12)
- U2 pad 13: Net-(U2-VDDA) -> /VDDA
- U2 pad 31: GND -> unconnected-(U2-VCAP_1-Pad31)
- U2 pad 44: ROW3 -> USB-D-
- U2 pad 45: ROW4 -> USB-D+
- U2 pad 46: ROW5 -> /TMS
- U2 pad 47: GND -> unconnected-(U2-VCAP_2-Pad47)
- U2 pad 49: ROW6 -> /TCK
Routing:
- net ROW6: track 74.3 -> 0.00 mm, vias 1 -> 0
- net /TCK: track 0.00 -> 72.0 mm, vias 0 -> 1
- net ROW4: track 70.6 -> 0.00 mm, vias 1 -> 0
- net ROW5: track 70.0 -> 0.00 mm, vias 1 -> 0
- net USB-D+: track 0.00 -> 65.4 mm, vias 0 -> 1
- net /TMS: track 0.00 -> 62.0 mm, vias 0 -> 1
- net /SCL1: track 0.00 -> 46.1 mm
- net /SDA1: track 0.00 -> 39.3 mm
- net Net-(U2-PH0): track 0.00 -> 20.5 mm
- net Net-(U2-PH1): track 0.00 -> 17.4 mm
- net /VDDA: track 0.00 -> 9.59 mm
- net COL0: track 65.5 -> 58.8 mm
- net ROW3: track 154.6 -> 148.6 mm
- net ROW2: track 163.8 -> 159.0 mm
- net ROW1: track 171.7 -> 167.7 mm
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Other:
- board size 113 x 101.1 mm -> 113 x 182.9 mm
