File: PCB-KiCAD/TeensyRPN42/leds.kicad_sch (KiCad schematic)
At the start: 2 parts

Commit message: more PCB
Parts:
- removed D1: SK6812MINI, LED_SMD:LED_SK6812MINI_PLCC4_3.5x3.5mm_P1.75mm, symbol LED:SK6812MINI
- added C14, C15, C16, C17, C18, C19, C20, C21, C22, C23, C24, C25: 100nF, Capacitor_SMD:C_0603_1608Metric_Pad1.08x0.95mm_HandSolder, symbol Device:C
- added D1, D10, D11, D12, D13, D14, D15, D16, D17, D18, D3, D4, D5, D6, D7, D8, D9: SK6805, LED_SMD:LED_SK6805_PLCC4_2.4x2.7mm_P1.3mm, symbol LED:SK6805
- added L3: L_Ferrite_Small, Inductor_SMD:L_0603_1608Metric_Pad1.05x0.95mm_HandSolder, symbol Device:L_Ferrite_Small
- added R2: 330, Resistor_SMD:R_0603_1608Metric_Pad0.98x0.95mm_HandSolder, symbol Device:R
- added U3: SN74LV1T125DBV, Package_TO_SOT_SMD:SOT-23-5, symbol Logic_LevelTranslator:SN74LV1T125DBV
Connections:
- net at D2.1 (DOUT): now also D3.3 (DIN)
- net GND: now reaches D2.2 (VSS)
- net GND: now also C14.2, C15.2, C16.2, C17.2, C18.2, C19.2, C20.2, C21.2, C22.2, C23.2, C24.2, C25.2, D1.2 (VSS), D10.2 (VSS), D11.2 (VSS), D12.2 (VSS), D13.2 (VSS), D14.2 (VSS), D15.2 (VSS), D16.2 (VSS), D17.2 (VSS), D18.2 (VSS), D3.2 (VSS), D4.2 (VSS), D5.2 (VSS), D6.2 (VSS), D7.2 (VSS), D8.2 (VSS), D9.2 (VSS), U3.1 (~{OE}), U3.3 (GND)
- net at D2.3 (DIN): now also D1.1 (DOUT)
- net V-LED: now reaches D2.4 (VDD)
- net V-LED: now also C14.1, C15.1, C16.1, C17.1, C18.1, C19.1, C20.1, C21.1, C22.1, C23.1, C24.1, C25.1, D1.4 (VDD), D10.4 (VDD), D11.4 (VDD), D12.4 (VDD), D13.4 (VDD), D14.4 (VDD), D15.4 (VDD), D16.4 (VDD), D17.4 (VDD), D18.4 (VDD), D3.4 (VDD), D4.4 (VDD), D5.4 (VDD), D6.4 (VDD), D7.4 (VDD), D8.4 (VDD), D9.4 (VDD), L3.2
- new net: D10.3 (DIN), D9.1 (DOUT)
- new net: D8.1 (DOUT), D9.3 (DIN)
- new net: D3.1 (DOUT), D4.3 (DIN)
- new net: D14.1 (DOUT), D15.3 (DIN)
- new net: D13.1 (DOUT), D14.3 (DIN)
- new net: R2.1, U3.4 (Y)
- new net: D1.3 (DIN), R2.2
- new net: D11.1 (DOUT), D12.3 (DIN)
- new net: D10.1 (DOUT), D11.3 (DIN)
- new net: D6.1 (DOUT), D7.3 (DIN)
- new net: D5.1 (DOUT), D6.3 (DIN)
- new net: D4.1 (DOUT), D5.3 (DIN)
- new net: D12.1 (DOUT), D13.3 (DIN)
- new net: D7.1 (DOUT), D8.3 (DIN)
- new net: D17.1 (DOUT), D18.3 (DIN)
- new net: D15.1 (DOUT), D16.3 (DIN)
- new net: D16.1 (DOUT), D17.3 (DIN)
- new net +5V: L3.1, U3.5 (VCC)
- new net LEDs: U3.2 (A)
Other:
- moved on the sheet: D2

Commit message: more pcb ...
Parts:
- U3: value SN74LV1T125DBV -> 74!AHCT!125; footprint Package_TO_SOT_SMD:SOT-23-5 -> Package_TO_SOT_SMD:SOT-353_SC-70-5; Reichelt (none) -> 74AHCT1G125GW
