File: PCB-KiCAD/TeensyRPN42/untitled.kicad_sch (KiCad schematic)
At the start: 41 parts, among them SW38 SW_DPST_x2, SW39 SW_DPST_x2, SW40 SW_DPST_x2, SW41 SW_DPST_x2, SW42 SW_DPST_x2, SW43 SW_DPST_x2, SW44 SW_DPST_x2, SW45 SW_DPST_x2, SW46 SW_DPST_x2, SW48 SW_DPST_x2, SW49 SW_DPST_x2, SW50 SW_DPST_x2, SW51 SW_DPST_x2, SW52 SW_DPST_x2, SW53 SW_DPST_x2, SW54 SW_DPST_x2, SW55 SW_DPST_x2, SW56 SW_DPST_x2, SW57 SW_DPST_x2, SW58 SW_DPST_x2, SW59 SW_DPST_x2, SW60 SW_DPST_x2, SW61 SW_DPST_x2, SW62 SW_DPST_x2, SW63 SW_DPST_x2, SW64 SW_DPST_x2, SW65 SW_DPST_x2, SW66 SW_DPST_x2, SW67 SW_DPST_x2, SW68 SW_DPST_x2, SW69 SW_DPST_x2, SW70 SW_DPST_x2, SW71 SW_DPST_x2, SW72 SW_DPST_x2, SW73 SW_DPST_x2, SW74 SW_DPST_x2, SW75 SW_DPST_x2, SW76 SW_DPST_x2, SW77 SW_DPST_x2, SW78 SW_DPST_x2, SW79 SW_DPST_x2

Commit message: A little PCBing
Parts:
- removed SW59, SW66, SW73, SW79: SW_DPST_x2, keyswitches:Kailh_socket_PG1350, symbol Switch:SW_DPST_x2
- added U1: HT1632C-52LQFP, Package_QFP:LQFP-52_14x14mm_P1mm, symbol Driver_LED:HT1632C-52LQFP
- SW38, SW39, SW40, SW41, SW42, SW43, SW44, SW45, SW48, SW49, SW50, SW51, SW52, SW58, SW61, SW62, SW63, SW64, SW65, SW68, SW69, SW70, SW71, SW72, SW75, SW76, SW77, SW78: footprint keyswitches:Kailh_socket_PG1350 -> PCM_Switch_Keyboard_Kailh:SW_Kailh_Choc_V1_1.00u
- SW46: footprint keyswitches:Kailh_socket_PG1350 -> PCM_Switch_Keyboard_Kailh:SW_Kailh_Choc_V1_2.00u
- SW53, SW54, SW55, SW56, SW57, SW60, SW67, SW74: footprint keyswitches:Kailh_socket_PG1350 -> PCM_Switch_Keyboard_Kailh:SW_Kailh_Choc_V1_1.25u
Connections:
- new net: U1.14 (VSS), U1.25 (VSS), U1.36 (VSS)
Other:
- moved on the sheet: SW38A, SW45A, SW51A, SW58A, SW65A, SW68A

Commit message: more PCB
Parts:
- removed U1: HT1632C-52LQFP, Package_QFP:LQFP-52_14x14mm_P1mm, symbol Driver_LED:HT1632C-52LQFP
- SW61, SW62, SW63, SW64, SW69, SW70, SW71, SW72, SW75, SW76, SW77, SW78: footprint PCM_Switch_Keyboard_Kailh:SW_Kailh_Choc_V1_1.00u -> PCM_Switch_Keyboard_Kailh:SW_Kailh_Choc_V1_1.25u
Connections:
- net ROW2: now reaches SW41.1 (A)
- net ROW2: now also SW39.1 (A), SW40.1 (A), SW42.1 (A), SW43.1 (A), SW44.1 (A)
- net ROW5: now reaches SW60.1 (A)
- net ROW5: now also SW61.1 (A), SW62.1 (A), SW63.1 (A), SW64.1 (A)
- net ROW7: now reaches SW74.1 (A)
- net ROW7: now also SW75.1 (A), SW76.1 (A), SW77.1 (A), SW78.1 (A)
- net ROW1: now reaches SW38.1 (A)
- net ROW1: now also SW45.1 (A), SW51.1 (A), SW58.1 (A), SW65.1 (A), SW68.1 (A)
- net COL0: now reaches SW38.2 (B)
- net ROW3: now reaches SW49.1 (A)
- net ROW3: now also SW46.1 (A), SW48.1 (A), SW50.1 (A), SW52.1 (A)
- net COL2: now reaches SW51.2 (B)
- net ROW4: now reaches SW56.1 (A)
- net ROW4: now also SW53.1 (A), SW54.1 (A), SW55.1 (A), SW57.1 (A)
- net ROW6: now reaches SW72.1 (A)
- net ROW6: now also SW67.1 (A), SW69.1 (A), SW70.1 (A), SW71.1 (A)
- net COL1: now reaches SW45.2 (B)
- net COL4: now reaches SW65.2 (B)
- net COL5: now reaches SW68.2 (B)
- net COL3: now reaches SW58.2 (B)
Other:
- note added: "Add Diodes ?"
- note added: "Dedicated Function Keys ???"
